File: Brainzy.brd (EAGLE design)
At the start: 100 x 100 mm, 78 parts, among them J7 5.5x2.1mm Barrel, Q1 BSS138, Q2 BSS138, Q3 BSS138, T1 BSS84, T2 BSS84, T3 BSS84, U1 L293DD, U2 L293DD, U3 HC_05

Commit message: Upload Brainzy v3.2
Parts:
- removed R27: 470, SparkFun-Resistors:1206
- added S1: (no value), SparkFun-Switches:SWITCH_SPST_SMD_A
- BATT: value BATTERY-CONNECTOR-LONG-PAD -> (none); device MrRobotics-Connectors:JST-XH-04-PACKAGE-LONG-PAD -> SparkFun-Connectors:1X04_LOCK_LONGPADS
- U$10, U$11, U$8, U$9: device holes:3,3 -> holes:4,3
- moved BATT 44.1 mm to (3.75, 42.2), flipped to the bottom, turned to 0 degrees
- moved PWR 28.3 mm to (-41.9, -19.5)
- moved ON/OFF 11.0 mm to (-35.1, 10.9), turned to 0 degrees
- moved R19 10.7 mm to (37.4, -23.0)
- moved LS1 7.25 mm to (-25.4, 0.00)
- moved D1 3.05 mm to (-9.25, -5.25)
- moved D3 2.81 mm to (9.25, -5.25)
- moved R5 2.50 mm to (-19.0, -30.9)
- moved R6 2.50 mm to (-16.5, -30.9)
- moved D2 1.25 mm to (0.00, 9.38)
- moved Q1 1.25 mm to (6.12, -15.4)
- moved Q2 1.25 mm to (-10.1, -15.4)
- moved Q3 1.25 mm to (-22.9, -15.4)
- moved R1 1.25 mm to (16.5, -21.9)
- moved R10 1.25 mm to (-13.9, -15.4)
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Connections:
- removed net BT_KEY: R27.2, U$1.3
- removed net N$8: LS1.+, U$1.29
- new net BUZZER: LS1.+, U$1.3
- net 3.3V: now also S1.1
- net 5V: now also MOT_FRONT.5, MOT_LEFT.5, MOT_RIGHT.5; no longer MOT_FRONT.3, MOT_LEFT.3, MOT_RIGHT.3
- net ENC1_A: now also MOT_LEFT.4; no longer MOT_LEFT.5
- net ENC1_B: now also MOT_LEFT.3; no longer MOT_LEFT.6
- net ENC2_A: now also MOT_RIGHT.4; no longer MOT_RIGHT.5
- net ENC2_B: now also MOT_RIGHT.3; no longer MOT_RIGHT.6
- net ENC3_A: now also MOT_FRONT.4, U$1.38/A19; no longer MOT_FRONT.5, U$1.37/A18
- net ENC3_B: now also MOT_FRONT.3, U$1.37/A18; no longer MOT_FRONT.6, U$1.38/A19
- net GND: now also MOT_FRONT.2, MOT_LEFT.2, MOT_RIGHT.2; no longer MOT_FRONT.4, MOT_LEFT.4, MOT_RIGHT.4
- net MOT1_OUT2: now also MOT_LEFT.6; no longer MOT_LEFT.2
- net MOT2_OUT2: now also MOT_RIGHT.6; no longer MOT_RIGHT.2
- net MOT3_OUT2: now also MOT_FRONT.6; no longer MOT_FRONT.2
- net N$18: now also S1.2, S1.3; no longer R27.1
Routing:
- net BUZZER: track 0.00 -> 50.3 mm
- net S1: track 76.3 -> 125.3 mm, vias 2 -> 3
- net S2: track 57.9 -> 106.8 mm, vias 2 -> 3
- net S3: track 43.8 -> 90.7 mm, vias 0 -> 1
- net I2C_SCL: track 190.7 -> 233.0 mm
- net I2C_SDA: track 210.9 -> 237.2 mm
- net 3.3V: track 112.6 -> 133.0 mm
- net TX5: track 53.7 -> 71.5 mm
- net 5V: track 392.4 -> 409.9 mm, vias 2 -> 4
- net N$18: track 23.7 -> 38.5 mm
- net BT_KEY: track 12.6 -> 0.00 mm
- net ENC2_A: track 72.9 -> 61.6 mm
- net N$8: track 9.93 -> 0.00 mm
- net MOT2_OUT2: track 14.8 -> 5.33 mm
- net N$15: track 28.7 -> 37.9 mm
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Other:
- board text added: "1"
- board text added: "2"
- board text added: "3"
- board text added: "4"
- board text added: "5"
- board text added: "6"
- board text added: "AT-MODE"
- board text added: "Brainzy v3.2"
- board text added: "OFF"
- board text added: "ON"
- board text removed: "Brainzy v3.1"

Commit message: Upload Brainzy v3.2.1
Parts:
- removed U$2: DC-DC-STEP-DOWN-MP2307_SMD, MrRobotics-Modules:DC-DC-STEP-DOWN-MP2307_SMD
- added BK: MP2307, SOIC127P600X170-9N:SOIC127P600X170-9N
- added C1, C2: 22uF, SparkFun-Capacitors:0805
- added C3: 0.1uF, SparkFun-Capacitors:0603
- added C4, C5: 10uF, SparkFun-Capacitors:1210
- added C6: 10nF, SparkFun-Capacitors:0603
- added C7: 3.3nF, SparkFun-Capacitors:0603
- added L1: 10UH, Seeed-Inductor-2016:SMD-2P-L6.0XW6.0XH3.0MM
- added R27: 6.8k, SparkFun-Resistors:0603
- added R37: 10k, SparkFun-Resistors:0603
- added R38: 44.2k, SparkFun-Resistors:0603
- added R39: 100k, SparkFun-Resistors:0603
- moved R20 22.0 mm to (-11.1, 13.9)
- turned D2 to 180 degrees
Connections:
- new net N$30: BK.5, R37.2, R38.1
- new net N$32: BK.8, C3.1
- new net N$33: BK.6, C7.1
- new net N$34: BK.3, C6.2, L1.2
- new net N$35: C7.2, R27.1
- new net N$36: BK.1, C6.1
- new net N$8: BK.7, R39.1
- net 12V: now also BK.2, C4.1, C5.1, R39.2; no longer U$2.IN+
- net 5V: now also C1.1, C2.1, L1.1, R38.2; no longer U$2.OUT+
- net GND: now also BK.4, BK.9, C1.2, C2.2, C3.2, C4.2, C5.2, R27.2, R37.1; no longer U$2.IN-, U$2.OUT-
Routing:
- net 12V: track 169.5 -> 185.0 mm, vias 2 -> 3
- net N$34: track 0.00 -> 11.1 mm
- net N$36: track 0.00 -> 10.4 mm, vias 0 -> 2
- net N$30: track 0.00 -> 4.96 mm
- net 5V: track 409.9 -> 406.3 mm
- net N$33: track 0.00 -> 3.52 mm
- net D3: track 49.4 -> 52.9 mm
- net N$8: track 0.00 -> 3.17 mm
- net N$35: track 0.00 -> 2.83 mm
- net N$32: track 0.00 -> 2.81 mm
