File: Brainzy.sch (EAGLE design)
At the start: 73 parts, among them J7 5.5x2.1mm Barrel, Q1 BSS138, Q2 BSS138, Q3 BSS138, Q4 BSS138, T1 BSS84, T2 BSS84, T3 BSS84, T4 SI2323DS, U1 L293DD, U2 L293DD, U3 HC_05, U4 GY-521MPU6050

Commit message: Upload Brainzy v3.0
Parts:
- removed C1, C2, C3, C4: 10uF, SparkFun-Capacitors:10UF-1206-6.3V-20%
- removed EXT_BT: (no value), SparkFun-Connectors:CONN_041X04_NO_SILK
- removed H1, H2, H3, H4: MOUNT-HOLE3.2, holes:MOUNT-HOLE3.2
- removed I2C1, I2C2, I2C3, UART: (no value), SparkFun-Connectors:CONN_04
- removed JP1: JUMPER-SMT_2_NO_NO-SILK, SparkFun-Jumpers:JUMPER-SMT_2_NO_NO-SILK
- removed S1: (no value), SparkFun-Switches:MOMENTARY-SWITCH-SPST-2-SMD-5.2MM
- removed SHARP1, SHARP2, SHARP3, SHARP4: (no value), SparkFun-Connectors:CONN_03
- removed SPI: (no value), MrRobotics-Connectors:CONN_05X2_EXTSHD_LOCK
- removed U$3: LOGO, MrRobotics-Aesthetics:LOGO
- removed U$4: LOGO_FR, MrRobotics-Aesthetics:LOGO_FR
- removed U4: GY-521MPU6050, MrRobotics-Modules:GY-521MPU6050
- removed UI: (no value), SparkFun-Connectors:CONN_04X2
- added D3: (no value), SparkFun-LED:LED-FKIT-1206
- added EXT1, EXT2, EXT3: (no value), SparkFun-Connectors:CONN_05X2SHD_LOCK
- added R26, R27: 470, SparkFun-Resistors:10OHM-1206-1/4W-1%
- added S4: (no value), SparkFun-Switches:MOMENTARY-SWITCH-SPST-2-SMD-5.2MM
- added SENSOR1, SENSOR2, SENSOR3, SENSOR4, SENSOR5, SENSOR6: (no value), MrRobotics-Connectors:JST-PH6
- R23: value 470k -> 150k
- R24: value 150k -> 470k
- R7: value 750 -> 470
Connections:
- net N$12 renamed PROG
- removed net BTN_CENTER: U$1.4/CAN0-RX/SDA2/PWM, UI.5
- removed net BTN_DOWN: U$1.7/RX3/PWM, UI.4
- removed net BTN_LEFT: U$1.3/CAN0-TX/SCL2/PWM, UI.3
- removed net BTN_RIGHT: U$1.5/PWM, UI.6
- removed net BTN_UP: U$1.2/PWM, UI.1
- removed net BT_RST: S3.1, U3.RST
- removed net DTR: U3.PIO9
- removed net EXT_RX: U$1.31/A12/RX4, UART.3
- removed net EXT_TX: U$1.32/A13/TX4/SCK1, UART.4
- removed net MPU_INT: U$1.26, U4.INT
- removed net N$17: JP1.1, U4.ADO
- removed net SHARP1: SHARP1.1, U$1.38/A19/SDA1/PWM
- removed net SHARP2: SHARP2.1, U$1.37/A18/SCL1/PWM
- removed net SHARP3: SHARP3.1, U$1.35/A16/PWM
- removed net SHARP4: SHARP4.1, U$1.36/A17/PWM
- new net BT_KEY: R27.2, U$1.3/CAN0-TX/SCL2/PWM
- new net EXT1_RX: EXT1.2, U$1.7/RX3/PWM
- new net EXT1_TX: EXT1.4, U$1.8/TX3/PWM
- new net EXT2_RX: EXT1.6, U$1.34/A15/RX5
- new net EXT2_TX: EXT1.8, U$1.33/A14/TX5
- new net LED_BUILDIN: R26.1, U$1.5/PWM
- new net N$12: D3.A, R26.2
- new net RST: S4.2, U$1.RST
- net 3.3V: no longer S1.3
- net 5V: now also EXT1.1, EXT2.1, EXT3.1, SENSOR1.6, SENSOR2.6, SENSOR3.6, SENSOR4.6, SENSOR5.6, SENSOR6.6; no longer C1.1, C2.1, C3.1, C4.1, EXT_BT.1, I2C1.2, I2C2.2, I2C3.2, JP1.2, SHARP1.3, SHARP2.3, SHARP3.3, SHARP4.3, SPI.1-VCC, U4.VCC, UART.2, UI.2
- net BATT1: now also U$1.A22/DAC1; no longer U$1.39/A20
- net BATT3: now also U$1.39/A20; no longer U$1.A22/DAC1
- net BT_RX: no longer EXT_BT.3
- net BT_TX: no longer EXT_BT.4
- net ENC1_B: now also MOT_LEFT.6-CHB, R1.1, U$1.21/A7/PWM; no longer U$1.17/A3/PWM
- net ENC2_A: now also U$1.2/PWM; no longer U$1.8/TX3/PWM
- net ENC2_B: no longer MOT_LEFT.6-CHB, R1.1
- net ENC3_A: now also U$1.37/A18/SCL1/PWM; no longer U$1.27
- net ENC3_B: now also U$1.38/A19/SDA1/PWM; no longer U$1.28
- net GND: now also D3.C, EXT1.9, EXT2.9, EXT3.9, S4.4, SENSOR1.1, SENSOR2.1, SENSOR3.1, SENSOR4.1, SENSOR5.1, SENSOR6.1; no longer C1.2, C2.2, C3.2, C4.2, EXT_BT.2, I2C1.1, I2C2.1, I2C3.1, S3.3, SHARP1.2, SHARP2.2, SHARP3.2, SHARP4.2, SPI.2-GND, U4.GND, UART.1, UI.8
- net I2C_SCL: now also EXT2.4, EXT2.8, SENSOR1.3, SENSOR2.3, SENSOR3.3, SENSOR4.3, SENSOR5.3, SENSOR6.3; no longer I2C1.4, I2C2.4, I2C3.4, U4.SCL
- net I2C_SDA: now also EXT2.2, EXT2.6, SENSOR1.4, SENSOR2.4, SENSOR3.4, SENSOR4.4, SENSOR5.4, SENSOR6.4; no longer I2C1.3, I2C2.3, I2C3.3, U4.SDA
- net MOT1_1: now also U$1.22/A8/PWM, U1.IN1; no longer U$1.23/A9/PWM, U1.IN2
- net MOT1_2: now also U$1.23/A9/PWM, U1.IN2; no longer U$1.22/A8/PWM, U1.IN1
- net MOT1_OUT1: now also U1.OUT1; no longer U1.OUT2
- net MOT1_OUT2: now also U1.OUT2; no longer U1.OUT1
- net MOT2_1: now also U$1.6/PWM, U1.IN4; no longer U$1.21/A7/PWM, U1.IN3
- net MOT2_2: now also U1.IN3; no longer U1.IN4
- net MOT2_OUT1: now also U1.OUT4; no longer U1.OUT3
- net MOT2_OUT2: now also U1.OUT3; no longer U1.OUT4
- net MOT3_1: now also U$1.35/A16/PWM, U2.IN4; no longer U$1.29/PWM, U2.IN3
- net MOT3_2: now also U$1.36/A17/PWM, U2.IN3; no longer U$1.30/PWM, U2.IN4
- net MOT3_OUT1: now also U2.OUT4; no longer U2.OUT3
- net MOT3_OUT2: now also U2.OUT3; no longer U2.OUT4
- net N$18: now also R27.1; no longer S1.1
- net N$8: now also U$1.29/PWM; no longer U$1.6/PWM
- net SPI_CS1: now also EXT3.2; no longer SPI.4-CS1
- net SPI_CS2: now also EXT3.4; no longer SPI.6-CS2
- net SPI_CS3: now also EXT3.6; no longer SPI.8-CS3
- net SPI_MISO: now also EXT3.5; no longer SPI.7-MISO
- net SPI_MOSI: now also EXT3.3; no longer SPI.5-MOSI
- net SPI_SCK: now also EXT3.8; no longer SPI.3-SCLK
- net T_CS: now also EXT3.7; no longer SPI.9-T_CS
- net T_IRQ: now also EXT3.10; no longer SPI.10-T_IRQ
- net WIFI_RX: now also U$1.31/A12/RX4; no longer U$1.34/A15/RX5
- net WIFI_TX: now also U$1.32/A13/TX4/SCK1; no longer U$1.33/A14/TX5
Other:
- note added: "Extension Inputs"
- note added: "Power"
- note added: "Sensor Inputs"
- note removed: "Extension for HC-05/06 breakout board"
- note removed: "I2C, SPI & UART Communications"
- note removed: "IR Range Sensors"
- note removed: "JP1 selects between I2C addresses 0x68 and 0x69"
- note removed: "Power Control"
- moved on the sheet: BUZZER, Q4, R18, R19, R22, R25, S3, U$2, U$6

Commit message: Upload Brainzy v3.1
Parts:
- removed BUZZER: (no value), MrRobotics-Components:BUZZER_MINI1X03_NO_SILK
- removed Q4: BSS138, MrRobotics-Transistors:BSS138
- removed S3, S4: (no value), SparkFun-Switches:MOMENTARY-SWITCH-SPST-2-SMD-5.2MM
- removed T4: SI2323DS, MrRobotics-Transistors:SI2323DS
- added LS1: BUZZER-PTH, SparkFun-Electromechanical:BUZZER-PTH
- added ON/OFF: JST-XH-02-PIN-LONG-PAD, MrRobotics-Connectors:JST-XH-02-PIN-LONG-PAD
- added PWR: JUMPER-SMT_2_NO_SILK, SparkFun-Jumpers:JUMPER-SMT_2_NO_SILK
- added R28, R29, R32, R33, R36: 150k, SparkFun-Resistors:10OHM-1206-1/4W-1%
- added R30, R31, R34, R35: 470k, SparkFun-Resistors:10OHM-1206-1/4W-1%
- added RST: MOMENTARY-SWITCH-SPST-PTH-6.0MM, SparkFun-Switches:MOMENTARY-SWITCH-SPST-PTH-6.0MM
- R21: value 470k -> 470
- S2: value (none) -> MOMENTARY-SWITCH-SPST-LED-PTH-12MM; device SparkFun-Switches:SWITCH-SPDT-SMD-RIGHT-ANGLE -> SparkFun-Switches:MOMENTARY-SWITCH-SPST-LED-PTH-12MM
- SENSOR1, SENSOR2, SENSOR3, SENSOR4, SENSOR5, SENSOR6: device MrRobotics-Connectors:JST-PH6 -> MrRobotics-Connectors:JST-ZH6
- U$1: value TEENSY_3.5-3.2INV -> TEENSY_3.5-3.2; device MrRobotics-Boards:TEENSY_3.5-3.2INV -> MrRobotics-Boards:TEENSY_3.5-3.2
Connections:
- net EXT2_RX renamed RX5
- net EXT2_TX renamed TX5
- net LED_BUILDIN renamed LED_BUILTIN
- net T_CS renamed D5
- net T_IRQ renamed D6
- removed net EXT1_RX: EXT1.2, U$1.7/RX3/PWM
- removed net EXT1_TX: EXT1.4, U$1.8/TX3/PWM
- removed net PROG: S3.2, U$1.PGM
- new net BTN_PROG: S2.1, U$1.4/CAN0-RX/SDA2/PWM
- new net D1: EXT1.5, U$1.28
- new net D2: EXT1.10, U$1.30/PWM
- new net D3: EXT2.5, U$1.26
- new net D4: EXT2.10, U$1.27
- new net LED_BTN_PROG: R21.1, U$1.17/A3/PWM
- new net N$17: SENSOR6.2, SENSOR6.5
- new net N$21: R28.1, SENSOR4.5
- new net N$22: R31.2, R32.2, SENSOR5.2
- new net N$23: R32.1, SENSOR5.5
- new net N$24: R29.2, R30.2, SENSOR2.2
- new net N$25: R30.1, SENSOR2.5
- new net N$26: R33.2, R35.2
- new net N$27: R34.2, R35.1, SENSOR3.2
- new net N$28: R33.1, SENSOR3.5
- new net N$29: R28.2, R36.2
- new net RX4: EXT1.2, U$1.31/A12/RX4
- new net TX4: EXT1.4, U$1.32/A13/TX4/SCK1
- new net WIFI_RST: U$6.RST
- net 12V: now also EXT1.3, EXT2.3, ON/OFF.2, PWR.2; no longer T4.D
- net 3.3V: no longer BUZZER.1
- net GND: now also EXT1.7, EXT2.7, LS1.2, R25.1, R29.1, R31.1, R34.1, RST.2, S2.2, S2.C, SENSOR1.2; no longer Q4.S, R25.2, S2.P, S2.S, S3.4, S4.4
- net N$15: now also ON/OFF.1, PWR.1; no longer R21.1, T4.S
- net N$16: now also S2.A; no longer S2.O, T4.G
- net N$20: now also R25.2, R36.1, SENSOR4.2; no longer BUZZER.3, Q4.D
- net N$8: now also LS1.1; no longer Q4.G, R25.1
- net RST: now also RST.1; no longer S4.2
- net WIFI_RX: now also U$1.7/RX3/PWM; no longer U$1.31/A12/RX4
- net WIFI_TX: now also U$1.8/TX3/PWM; no longer U$1.32/A13/TX4/SCK1
Other:
- moved on the sheet: D3, R22, R25, R26

Commit message: Upload Brainzy v3.2
Parts:
- removed R27: 470, SparkFun-Resistors:10OHM-1206-1/4W-1%
- added S1: (no value), SparkFun-Switches:SWITCH-SPDT-SMD-RIGHT-ANGLE
- BATT: value BATTERY-CONNECTOR-LONG-PAD -> (none); device MrRobotics-Connectors:BATTERY-CONNECTOR-LONG-PAD -> SparkFun-Connectors:CONN_04LOCK_LONGPADS
Connections:
- removed net BT_KEY: R27.2, U$1.3/CAN0-TX/SCL2/PWM
- removed net N$8: LS1.1, U$1.29/PWM
- new net BUZZER: LS1.1, U$1.3/CAN0-TX/SCL2/PWM
- net 3.3V: now also S1.O
- net 5V: now also MOT_FRONT.5-CHA, MOT_LEFT.5-CHA, MOT_RIGHT.5-CHA; no longer MOT_FRONT.3-VCC, MOT_LEFT.3-VCC, MOT_RIGHT.3-VCC
- net ENC1_A: now also MOT_LEFT.4-GND; no longer MOT_LEFT.5-CHA
- net ENC1_B: now also MOT_LEFT.3-VCC; no longer MOT_LEFT.6-CHB
- net ENC2_A: now also MOT_RIGHT.4-GND; no longer MOT_RIGHT.5-CHA
- net ENC2_B: now also MOT_RIGHT.3-VCC; no longer MOT_RIGHT.6-CHB
- net ENC3_A: now also MOT_FRONT.4-GND, U$1.38/A19/SDA1/PWM; no longer MOT_FRONT.5-CHA, U$1.37/A18/SCL1/PWM
- net ENC3_B: now also MOT_FRONT.3-VCC, U$1.37/A18/SCL1/PWM; no longer MOT_FRONT.6-CHB, U$1.38/A19/SDA1/PWM
- net GND: now also BATT.1, MOT_FRONT.2-M+, MOT_LEFT.2-M+, MOT_RIGHT.2-M+; no longer BATT.1-GND, MOT_FRONT.4-GND, MOT_LEFT.4-GND, MOT_RIGHT.4-GND
- net MOT1_OUT2: now also MOT_LEFT.6-CHB; no longer MOT_LEFT.2-M+
- net MOT2_OUT2: now also MOT_RIGHT.6-CHB; no longer MOT_RIGHT.2-M+
- net MOT3_OUT2: now also MOT_FRONT.6-CHB; no longer MOT_FRONT.2-M+
- net N$18: now also S1.P, S1.S; no longer R27.1
- net S1: now also BATT.2; no longer BATT.2-S1
- net S2: now also BATT.3; no longer BATT.3-S2
- net S3: now also BATT.4; no longer BATT.4-S3
Other:
- moved on the sheet: LS1, R1, R19, R2, R3, R4, R5, R6

Commit message: Upload Brainzy v3.2.1
Parts:
- removed U$2: DC-DC-STEP-DOWN-MP2307_SMD, MrRobotics-Modules:DC-DC-STEP-DOWN-MP2307_SMD
- added BK: MP2307, SOIC127P600X170-9N:MP2307
- added C1, C2: 22uF, SparkFun-Capacitors:22UF-0805-6.3V-20%
- added C3: 0.1uF, SparkFun-Capacitors:0.1UF-0603-25V-5%
- added C4, C5: 10uF, SparkFun-Capacitors:10UF-1210-50V-20%
- added C6: 10nF, SparkFun-Capacitors:10NF-0603-50V-10%
- added C7: 3.3nF, SparkFun-Capacitors:3.3NF-0603-100V-10%
- added L1: 10UH, Seeed-Inductor-2016:SMD-INDUCTOR-10UH-20%(2P-6X6MM)'0630'
- added R27: 6.8k, SparkFun-Resistors:6.8KOHM-0603-1/10W-1%
- added R37: 10k, SparkFun-Resistors:10KOHM-0603-1/10W-1%
- added R38: 44.2k, SparkFun-Resistors:43KOHM-0603-1/10W-1%
- added R39: 100k, SparkFun-Resistors:100KOHM-0603-1/10W-1%
Connections:
- new net N$30: BK.P$5, R37.2, R38.1
- new net N$32: BK.P$8, C3.1
- new net N$33: BK.P$6, C7.1
- new net N$34: BK.P$3, C6.2, L1.2
- new net N$35: C7.2, R27.1
- new net N$36: BK.P$1, C6.1
- new net N$8: BK.P$7, R39.1
- net 12V: now also BK.P$2, C4.1, C5.1, R39.2; no longer U$2.IN+
- net 5V: now also C1.1, C2.1, L1.1, R38.2; no longer U$2.OUT+
- net GND: now also BK.P$4, C1.2, C2.2, C3.2, C4.2, C5.2, R27.2, R37.1; no longer U$2.IN-, U$2.OUT-
Other:
- note added: "Battery"
- note added: "Step-down converter"
- note removed: "Power"
